File: ledcube8x8x8-board.kicad_pcb (KiCad board)
At the start: 4 copper layers, 112.5 x 79.2 mm, 224 parts, among them J1 282836-2, J10 molex_53261-0871, J11 104031-0811, J12 30306-6002HB, J13 hedear, J14 hedear, J15 30306-6002HB, J16 61201021621, J2 molex_53261-0871, J3 molex_53261-0871, J4 molex_53261-0871, J5 molex_53261-0871, J6 molex_53261-0871, J7 molex_53261-0871, J8 molex_53261-0871, J9 molex_53261-0871, Q1 Q_NMOS_GDSD, Q10 Q_PMOS_GSD, Q2 Q_NMOS_GDSD, Q3 Q_NMOS_GDSD, Q4 Q_NMOS_GDSD, Q5 Q_NMOS_GDSD, Q6 Q_NMOS_GDSD, Q7 Q_NMOS_GDSD, Q8 Q_NMOS_GDSD, Q9 Q_PMOS_GSD, U1 LM1085IS-12, U10 TL3305AF260QG, U11 IP4220CZ6, U12 IP4220CZ6, U13 XC9572XL-VQ64, U14 SN74LVCC3245APWR, U15 SN74LVCC3245APWR, U16 TS3A27518EPW, U2 STP08CP05MTR, U3 STP08CP05MTR, U4 STP08CP05MTR, U5 STP08CP05MTR, U6 STP08CP05MTR, U7 STP08CP05MTR, U8 STP08CP05MTR, U9 STP08CP05MTR, X1 ASE-40MHz, X2 ASE-25MHz

Commit message: PCB complete
Parts:
- added NT10: Net-Tie_2, NetTie:NetTie-2_SMD_Pad0.5mm, F.Cu at (30.8, 21.5)
- added NT11: Net-Tie_2, NetTie:NetTie-2_SMD_Pad0.5mm, B.Cu at (105.8, 52.8)
- added NT12: Net-Tie_2, NetTie:NetTie-2_SMD_Pad0.5mm, F.Cu at (6.50, 35.2)
- moved U13 145.0 mm to (60.8, 48.2), turned to 0 degrees
- moved Q9 138.9 mm to (45.4, 57.9)
- moved R123 138.9 mm to (45.2, 54.0)
- moved R124 138.9 mm to (41.5, 58.0)
- moved C25 114.7 mm to (49.2, 56.5), turned to 270 degrees
- moved C20 108.3 mm to (52.5, 56.5), turned to 270 degrees
- moved C30 106.7 mm to (72.5, 45.5)
- moved C31 106.7 mm to (75.8, 45.5)
- moved C26 103.2 mm to (62.0, 36.8), turned to 90 degrees
- moved C27 96.8 mm to (65.2, 36.8), turned to 90 degrees
- moved C28 96.0 mm to (64.2, 58.5)
- moved C29 96.0 mm to (67.5, 58.5)
- moved C19 85.5 mm to (47.2, 45.5), turned to 270 degrees
- moved X2 81.8 mm to (50.9, 45.5), turned to 270 degrees
- moved C18 80.3 mm to (47.2, 50.2), turned to 270 degrees
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Connections:
- net /pl.sch/VCC_3V3 renamed /VCC_3V3
- net /pl.sch/VCC_5V0 renamed /VCC_5V0
- D6 pad 1: /power_supply.sch/~SYS_RST -> /pl.sch/~SYS_RST
- Q10 pad 1: /power_supply.sch/~SYS_RST -> /pl.sch/~SYS_RST
- R106 pad 1: /power_supply.sch/~SYS_RST -> /pl.sch/~SYS_RST
Routing:
- net /VCC_3V3: track 214.5 -> 486.0 mm, vias 1 -> 11
- net GNDD: track 294.7 -> 530.3 mm, vias 11 -> 33
- net GND: track 475.7 -> 677.6 mm, vias 49 -> 76
- net /pl.sch/~SYS_RST: track 2.97 -> 185.9 mm, vias 0 -> 5
- net /power_supply.sch/~SYS_RST: track 115.3 -> 0.00 mm, vias 3 -> 0
- net /pl.sch/LED_R: track 0.00 -> 55.6 mm, vias 0 -> 3
- net /pl.sch/LED_G: track 0.00 -> 51.4 mm, vias 0 -> 3
- net /LAYER_SEL5: track 0.00 -> 49.1 mm, vias 0 -> 1
- net /pl.sch/LED_O1: track 0.00 -> 47.1 mm, vias 0 -> 3
- net /LAYER_SEL7: track 0.00 -> 44.9 mm, vias 0 -> 1
- net /pl.sch/LED_O2: track 0.00 -> 44.3 mm, vias 0 -> 3
- net /LAYER_SEL8: track 0.00 -> 44.0 mm
- net /LAYER_SEL6: track 0.00 -> 43.7 mm, vias 0 -> 2
- net /ps.sch/MUX_SEL_PRG: track 23.1 -> 66.7 mm, vias 2 -> 5
- net /pl.sch/DATA_ROW6_3V3: track 0.00 -> 41.9 mm
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- added copper zone on B.Cu, net (none)
- added copper zone on F.Cu, net (none)
Other:
- outline, holes or cut-outs redrawn
